File: Hardware/DiyMKbd.sch (EAGLE design)
At the start: 68 parts

Commit message: add gerber file
Parts:
- J1: value (none) -> 2.54 header
Changed lines of the file:
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@@
 <part name="GND1" library="supply1" deviceset="GND" device=""/>
 <part name="GND2" library="supply1" deviceset="GND" device=""/>
-<part name="J1" library="SparkFun-Connectors" deviceset="CONN_03" device="LOCK"/>
+<part name="J1" library="SparkFun-Connectors" deviceset="CONN_03" device="LOCK" value="2.54 header"/>
 <part name="TP1" library="SparkFun-Connectors" deviceset="TEST-POINT" device="TP_15TH_THRU"/>
 <part name="FRAME1" library="SparkFun-Aesthetics" deviceset="FRAME-A4L" device=""/>
@@
 </sheet>
 </sheets>
+<errors>
+</errors>
 </schematic>
 </drawing>
